File: RadioMusicHardware/RadioMusic_F.sch (EAGLE design)
At the start: 30 parts, among them X1 VERT_SD_CARD_REV2

Commit message: starting SMD needs layout
Parts:
- removed C1: 100uf, gm-caps-electro-pol:050
- removed JP2: M11PTH, SparkFun-Connectors:M11PTH
- removed JP4: (no value), SparkFun-Connectors:M07
- added C3, C5, C8: 0.1uF, SparkFun-Capacitors:0.1UF-25V(+80/-20%)(0603)
- added C4: 10uf, rcl:CPOL-USB
- added C6, C7: 10uf, SparkFun-Passives:CAP_POLC
- added C9: 100u, SparkFun-Passives:CAP_POLC
- added D1, D2: DIODE-SCHOTTKY_, SparkFun-DiscreteSemi:DIODE-SCHOTTKY_
- added D3: (no value), SparkFun-DiscreteSemi:BAV99
- added IC2: 5v regulator, burr-brown:REG1117
- added R1, R6: 39k, SparkFun-Passives:RESISTOR0603-RES
- added R4: 5.6k, SparkFun-Passives:RESISTOR0603-RES
- added SV1: EURO_POWER_HEADERLOCK_PADS, MusicThingModular:EURO_POWER_HEADERLOCK_PADS
- added U1: TEENSY_3.1_TW, TomW:TEENSY_3.1_TW
- added U2: MCP6002, MusicThingModular:TL072_SMD
- added U3: TL072_SMD, MusicThingModular:TL072_SMD
- C2: value 100n -> 0.1uF; device TomW:C-EU050-024X044 -> SparkFun-Capacitors:0.1UF-25V(+80/-20%)(0603)
- R10, R13, R20, R21: device MusicThingModular:RESISTORVERTICAL -> SparkFun-Passives:RESISTOR0603-RES
- R11, R12, R14, R15, R17, R18, R19, R8, R9: device MusicThingModular:RESISTOR7MM -> SparkFun-Passives:RESISTOR0603-RES
Connections:
- new net +12V: C5.1, C6.+, D1.C, IC2.VIN, U3P.V+
- new net +3.3V: D3.C2, U1.3.3V, U2P.V+
- new net +5V: IC2.VOUT, U1.VIN
- new net -12V: C7.-, C8.2, D2.A, U3P.V-
- new net AUDIO_OUT: C3.2, R6.2, U3A.OUT
- new net CHANNEL_CV: U2A.+IN
- new net CHANNEL_POT: U1.23/A9
- new net DAC: C4.+, U1.DAC
- new net GND: C5.2, C6.-, C7.+, C8.1, D3.A1, IC2.GND, SV1.3, SV1.4, SV1.5, SV1.6, SV1.7, SV1.8, U1.AGND, U1.GND, U2P.V-, U3A.+IN, U3B.+IN
- new net LED1: U1.3
- new net LED2: U1.4
- new net LED3: U1.5
- new net LED4: U1.6
- new net LED_RESET: U1.11
- new net MISO: U1.12
- new net MOSI: U1.7
- new net N$4: C4.-, R1.2, R4.1
- new net N$5: C3.1, R4.2, R6.1, U3A.-IN
- new net N$7: U3B.-IN, U3B.OUT
- new net N$8: D1.A, SV1.10, SV1.9
- new net N$9: D2.C, SV1.1, SV1.2
- new net PIN20/A6: U1.20/A6, U2B.-IN, U2B.OUT
- new net PIN22/A8: U1.22/A8, U2A.-IN, U2A.OUT
- new net RESET_CV: D3.COM, U1.9
- new net RESET_SW: U1.8
- new net SCLK: U1.14/A0
- new net SS: U1.10
- new net TIME_CV: U2B.+IN
- new net TIME_POT: U1.21/A7
- net +3.3V_F: now also C9.+; no longer C1.+, JP4.4
- net AUDIO_OUT_F: no longer JP4.5
- net CHANNEL_CV_F: no longer JP4.6
- net CHANNEL_POT_F: no longer JP4.1
- net GND_F: now also C9.-; no longer C1.-, JP2.1
- net LED1_F: no longer JP2.2
- net LED2_F: no longer JP2.3
- net LED3_F: no longer JP2.4
- net LED4_F: no longer JP2.5
- net LED_RESET_F: no longer JP2.10
- net MISO_F: no longer JP2.11
- net MOSI_F: no longer JP2.6
- net RESET_CV_F: no longer JP2.8
- net RESET_SW_F: no longer JP2.7
- net SCLK_F: no longer JP4.3
- net SS_F: no longer JP2.9
- net TIME_CV_F: no longer JP4.7
- net TIME_POT_F: no longer JP4.2
Other:
- note added: "BACK = power/teensy FRONT = knobs & sockets Front Board requirements: +3.3v for pots & SD Card GND LED1 LED2 LED3 LED4 LEDReset Reset Button Reset CV Time CV Time Pot ChannelCV Channel Pot SD - MISO SD- MOSI SD-CLOCK SD-SS"
- note added: "SD Card Connections: SCLK 14 MISO 12 MOSI 7 SS 10"
- moved on the sheet: C2

Commit message: everything fits on the board, but not properly placed or routed
Parts:
- renumbered IC2 to REG1117
Changed lines of the file:
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@@
 <part name="D2" library="SparkFun-DiscreteSemi" deviceset="DIODE-SCHOTTKY" device="_"/>
 <part name="C9" library="SparkFun-Passives" deviceset="CAP_POL" device="C" value="100u"/>
-<part name="IC2" library="burr-brown" deviceset="REG1117" device="" value="5v regulator"/>
+<part name="REG1117" library="burr-brown" deviceset="REG1117" device="" value="5v regulator"/>
 <part name="D3" library="SparkFun-DiscreteSemi" deviceset="BAV99" device=""/>
 </parts>
@@
 <instance part="D2" gate="G$1" x="266.7" y="5.08"/>
 <instance part="C9" gate="G$1" x="132.08" y="121.92"/>
-<instance part="IC2" gate="G$1" x="365.76" y="30.48"/>
+<instance part="REG1117" gate="G$1" x="365.76" y="30.48"/>
 <instance part="D3" gate="G$1" x="345.44" y="91.44" rot="R90"/>
 </instances>
@@
 <wire x1="365.76" y1="17.78" x2="365.76" y2="15.24" width="0.1524" layer="91"/>
 <junction x="365.76" y="15.24"/>
-<pinref part="IC2" gate="G$1" pin="GND"/>
+<pinref part="REG1117" gate="G$1" pin="GND"/>
 </segment>
 <segment>
@@
 <wire x1="330.2" y1="30.48" x2="337.82" y2="30.48" width="0.1524" layer="91"/>
 <pinref part="U3" gate="P" pin="V+"/>
-<pinref part="IC2" gate="G$1" pin="VIN"/>
+<pinref part="REG1117" gate="G$1" pin="VIN"/>
 </segment>
 <segment>
@@
 <wire x1="381" y1="25.4" x2="378.46" y2="30.48" width="0.1524" layer="91"/>
 <label x="381" y="25.4" size="1.778" layer="95" xref="yes"/>
-<pinref part="IC2" gate="G$1" pin="VOUT"/>
-</segment>
-<segment>
+<pinref part="REG1117" gate="G$1" pin="VOUT"/>
+</segment>
+<segment>
